File: m0116_usb.kicad_pcb (KiCad board)
At the start: 2 copper layers, 372.1 x 113.8 mm, 186 parts, among them J1 AVR-ISP-6, J2 Conn_01x04, J3 Conn_01x04, U1 ATmega32A-PU

Commit message: Convert KiCad 5 project to KiCad 7 format
Pure format migration, no circuit or layout changes:

- m0116_usb.kicad_pcb: re-saved with KiCad 7.0.11 (186 footprints,
  843 segments, 4 vias, 126 nets, 3 zones preserved). Legacy zone fill
  strategy converted on a best-effort basis; zones need a refill
  before fabrication.
- m0116_usb.sch -> m0116_usb.kicad_sch, m0116_usb.pro ->
  m0116_usb.kicad_pro (net classes and design rules migrated).
- Symbols that differ from the KiCad 7 libraries (ATmega32A-PU, CP1,
  USB_B_Mini) were rescued into m0116_usb-rescue.kicad_sym.
- Removed legacy files (.sch, .pro, -cache.lib, -bak) and the local
  fp-info-cache; added .gitignore for KiCad per-user state.

Schematic netlist verified against PCB connectivity: all 120 multi-pin
nets match. The pre-existing reference mismatch Boot1/Reset1
(schematic) vs. Boot/Reset (PCB) is carried over unchanged.

Co-Authored-By: Claude Opus 5.5 <noreply@anthropic.com>
Other:
- net class Default removed
- net class Power removed

Commit message: Update PCB from schematic for the nice!nano controller
Generated with `make pcb-update`:

- removed the 20 footprints of the ATmega/V-USB controller
- added 32 footprints linked to the new symbols; 29 placed in the rear
  strip behind the number row, J4/R4/R5 parked above the board until
  the daughterboard tab is resized
- removed 377 track segments of vanished nets and 118 dangling stubs
- matrix tracks moved to the KiCad 7 net names (179 items)
- keepout (no tracks, vias, pour) under the nice!nano antenna
- zones refilled

Matrix footprints and pads are unchanged; all matrix nets remain fully
routed. 48 nets with new controller connections are still unrouted.

Co-Authored-By: Claude Opus 5.5 <noreply@anthropic.com>
Parts:
- removed Boot: Boot, Button_Switch_THT:SW_PUSH_6mm
- removed D1, D2: 3.6V, Diode_THT:D_DO-35_SOD27_P7.62mm_Horizontal
- removed F1: 500mA, Fuse:Fuse_Littelfuse_395Series
- removed Reset: Reset, Button_Switch_THT:SW_PUSH_6mm
- removed USB1: USB_B_Mini, random-keyboard-parts:Molex-0548190519
- removed XTAL1: Crystal, Crystal:Crystal_HC49-4H_Vertical
- added C6: 10u, Capacitor_THT:C_Disc_D5.0mm_W2.5mm_P5.00mm, F.Cu at (332.5, 81.5)
- added C7: 100n, Capacitor_THT:C_Disc_D3.0mm_W2.0mm_P2.50mm, F.Cu at (340.8, 81.5)
- added J4: USB-C (to nice!nano), Connector_USB:USB_C_Receptacle_GCT_USB4085, F.Cu at (27.0, 52.6)
- added JP1: SR_SUPPLY, Jumper:SolderJumper-3_P1.3mm_Bridged12_RoundedPad1.0x1.5mm_NumberLabels, F.Cu at (116.0, 88.5)
- added R5: 5k1, Resistor_THT:R_Axial_DIN0207_L6.3mm_D2.5mm_P2.54mm_Vertical, F.Cu at (58.7, 55.0)
- added SW1: Reset, Button_Switch_THT:SW_PUSH_6mm, F.Cu at (115.3, 76.8)
- added SW2: Battery, Button_Switch_THT:SW_Slide_SPDT_Angled_CK_OS102011MA1Q, F.Cu at (77.0, 80.0)
- added TP1: BAT_IN, TestPoint:TestPoint_THTPad_D1.5mm_Drill0.7mm, F.Cu at (64.8, 80.5)
- added TP2: VBAT, TestPoint:TestPoint_THTPad_D1.5mm_Drill0.7mm, F.Cu at (64.8, 84.0)
- added TP3: 3V3_AON, TestPoint:TestPoint_THTPad_D1.5mm_Drill0.7mm, F.Cu at (64.8, 87.5)
- added TP4: TP_PWR, TestPoint:TestPoint_THTPad_D1.5mm_Drill0.7mm, F.Cu at (346.5, 79.5)
- added TP5: TP_CLK, TestPoint:TestPoint_THTPad_D1.5mm_Drill0.7mm, F.Cu at (350.5, 79.5)
- added TP6: TP_DATA, TestPoint:TestPoint_THTPad_D1.5mm_Drill0.7mm, F.Cu at (346.5, 83.5)
- added TP7: GND, TestPoint:TestPoint_THTPad_D1.5mm_Drill0.7mm, F.Cu at (350.5, 83.5)
- added TP8: 3V3_SR, TestPoint:TestPoint_THTPad_D1.5mm_Drill0.7mm, F.Cu at (122.5, 88.5)
- added U2: 74HC595, Package_DIP:DIP-16_W7.62mm_Socket, F.Cu at (223.1, 83.8)
- added U3: 74HC595, Package_DIP:DIP-16_W7.62mm_Socket, F.Cu at (248.1, 83.8)
- added U4: 74HC595, Package_DIP:DIP-16_W7.62mm_Socket, F.Cu at (273.1, 83.8)
- added U5: MCP1700-3302E/TO, Package_TO_SOT_THT:TO-92_Inline, F.Cu at (86.7, 86.0)
- C1: value 4.7u -> 1u; footprint Capacitor_THT:CP_Radial_D5.0mm_P2.50mm -> Capacitor_THT:C_Disc_D3.0mm_W2.0mm_P2.50mm
- C2: value 0.1u -> 1u
- C3: value 0.1u -> 100n
- C4, C5: value 22p -> 100n; footprint Capacitor_THT:C_Disc_D6.0mm_W2.5mm_P5.00mm -> Capacitor_THT:C_Disc_D3.0mm_W2.0mm_P2.50mm
- J1: value AVR-ISP-6 -> LiPo; footprint Connector_PinHeader_2.54mm:PinHeader_2x03_P2.54mm_Horizontal -> Connector_JST:JST_PH_S2B-PH-K_1x02_P2.00mm_Horizontal
- J2: value Conn_01x04 -> TrackPoint; footprint Connector_PinHeader_2.00mm:PinHeader_1x04_P2.00mm_Vertical -> Connector_PinHeader_2.54mm:PinHeader_1x10_P2.54mm_Vertical
- J3: value Conn_01x04 -> USB-C (case); footprint Connector_JST:JST_PH_S4B-PH-K_1x04_P2.00mm_Horizontal -> Connector_USB:USB_C_Receptacle_GCT_USB4085
- R1: value 10k -> 4k7
- R2: value 1.5k -> 4k7
- R3: value 68R -> 100k
- R4: value 68R -> 5k1; footprint Resistor_THT:R_Axial_DIN0207_L6.3mm_D2.5mm_P10.16mm_Horizontal -> Resistor_THT:R_Axial_DIN0207_L6.3mm_D2.5mm_P2.54mm_Vertical
- U1: value ATmega32A-PU -> nice!nano_v2; footprint Package_DIP:DIP-40_W15.24mm_Socket -> Package_DIP:DIP-24_W15.24mm_Socket
- moved J1 272.9 mm to (69.0, 84.0), turned to 0 degrees
- moved J2 272.0 mm to (331.1, 88.5), turned to 90 degrees
- moved C2 184.9 mm to (91.8, 89.5), turned to 0 degrees
- moved R4 150.5 mm to (43.7, 55.0), turned to 0 degrees
- moved U1 136.9 mm to (167.0, 90.2), turned to 90 degrees
- moved R3 118.5 mm to (304.0, 87.7)
- moved R2 105.1 mm to (300.0, 87.7), turned to 90 degrees
- moved R1 66.1 mm to (296.0, 87.7)
- moved C3 52.1 mm to (230.8, 89.5), turned to 0 degrees
- moved C5 30.1 mm to (280.8, 89.5), turned to 0 degrees
- moved J3 19.2 mm to (51.7, 74.6), turned to 0 degrees
- moved C4 14.2 mm to (255.8, 89.5), turned to 0 degrees
- moved C1 10.6 mm to (81.8, 89.5), turned to 0 degrees
Connections:
- C1 pad 1: +5V -> /Controller/VBAT
- C2 pad 1: +5V -> /Controller/3V3_AON
- C3 pad 1: +5V -> /Controller/3V3_SR
- C4 pad 1: Net-(C4-Pad1) -> /Controller/3V3_SR
- C5 pad 1: Net-(C5-Pad1) -> /Controller/3V3_SR
- J1 pad 1: MISO -> /Controller/BAT_IN
- J1 pad 2: +5V -> GND
- J2 pad 1: VCC -> /Controller/TP_PWR
- J2 pad 2: Net-(J2-Pad2) -> GND
- J2 pad 3: Net-(J2-Pad3) -> /Controller/TP_CLK
- J2 pad 4: GND -> /Controller/TP_DATA
- R1 pad 1: +5V -> /Controller/TP_PWR
- R1 pad 2: reset -> /Controller/TP_CLK
- R2 pad 1: Net-(D2-Pad1) -> /Controller/TP_PWR
- R2 pad 2: +5V -> /Controller/TP_DATA
- R3 pad 1: Net-(D1-Pad1) -> /Controller/TP_RESET
- R3 pad 2: D+ -> GND
- R4 pad 1: Net-(D2-Pad1) -> /USB daughterboard/DB_CC1
- R4 pad 2: D- -> /USB daughterboard/DB_GND
- U1 pad 1: Net-(U1-Pad1) -> /Controller/TP_CLK
- U1 pad 10: +5V -> /Controller/TP_BTN_M
- U1 pad 11: GND -> /Controller/TP_BTN_R
- U1 pad 12: Net-(C5-Pad1) -> /Controller/TP_AUX1
- U1 pad 13: Net-(C4-Pad1) -> unconnected-(U1-P0.09/NFC1-Pad13)
- U1 pad 14: col4 -> /Controller/TP_AUX2
- U1 pad 15: col3 -> unconnected-(U1-P1.11-Pad15)
- U1 pad 16: D+ -> row4
- U1 pad 17: D- -> row3
- U1 pad 18: boot -> row2
- U1 pad 19: col2 -> row1
- U1 pad 2: row0 -> /Controller/TP_DATA
- U1 pad 20: col1 -> row0
- U1 pad 21: col5 -> /Controller/TP_PWR
- U1 pad 22: col6 -> /Controller/NRST
- U1 pad 23: col7 -> GND
- U1 pad 24: col8 -> /Controller/VBAT
- U1 pad 3: row1 -> GND
- U1 pad 4: Net-(U1-Pad4) -> GND
- U1 pad 5: Net-(U1-Pad5) -> /Controller/SR_DATA
- U1 pad 6: MOSI -> /Controller/SR_CLK
- U1 pad 7: MISO -> /Controller/SR_LATCH
- U1 pad 8: SCK -> /Controller/TP_RESET
- U1 pad 9: reset -> /Controller/TP_BTN_L
Routing:
- net +5V: track 353.9 -> 0.00 mm
- net col1: track 315.8 -> 76.3 mm
- net col2: track 309.7 -> 88.7 mm
- net col3: track 294.4 -> 83.1 mm
- net col4: track 275.2 -> 80.3 mm
- net reset: track 152.2 -> 0.00 mm
- net col5: track 206.2 -> 57.2 mm
- net Net-(D2-Pad1): track 144.4 -> 0.00 mm
- net col6: track 215.7 -> 83.1 mm
- net Net-(D1-Pad1): track 130.4 -> 0.00 mm
- net col7: track 173.6 -> 57.3 mm
- net col18: track 176.8 -> 68.7 mm
- net col17: track 159.5 -> 70.5 mm
- net col9: track 163.6 -> 78.3 mm
- net D-: track 83.2 -> 0.00 mm
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
Commit message: Add MX/Alps hybrid footprints, TKL variant and Freerouting workflow
Snapshot, routing still in progress.

- switch footprints changed to MX_Alps_Hybrid:MX-1U-NoLED, optional
  centred MX spacebar switch MX82
- m0116_tkl: board without keypad, generated by make tkl-sch / tkl-pcb,
  right edge copies the original contour; partially autorouted
  (open: col2, GND islands near U2/U3, USB daughterboard by hand)
- tools/export_matrix_dsn.py, tools/import_ses.py: Specctra DSN/SES
  round trip for Freerouting (make dsn, make dsn-continue)
- full board: old matrix tracks still cross the MX centre holes until
  it is rerouted

Co-Authored-By: Claude Opus 5.5 <noreply@anthropic.com>
Parts:
- added MX82: MX-NoLED, MX_Alps_Hybrid:MX-1U-NoLED, F.Cu at (160.4, 178.9)
- MX1, MX10, MX11, MX12, MX13, MX14, MX15, MX16, MX17, MX18, MX19, MX2, MX20, MX21, MX22, MX23, MX24, MX25, MX26, MX27, MX28, MX29, MX3, MX30, MX31, MX32, MX33, MX34, MX35, MX36, MX37, MX38, MX39, MX4, MX40, MX41, MX42, MX43, MX44, MX45, MX46, MX47, MX48, MX49, MX5, MX50, MX51, MX52, MX53, MX54, MX55, MX56, MX57, MX58, MX59, MX6, MX60, MX61, MX62, MX63, MX64, MX65, MX66, MX67, MX68, MX69, MX7, MX70, MX71, MX72, MX73, MX74, MX75, MX76, MX77, MX78, MX79, MX8, MX80, MX81, MX9: footprint Alps_Only:ALPS-1U -> MX_Alps_Hybrid:MX-1U-NoLED
Connections:
- net Net-(D75-A) renamed /SPACE_SW
