File: m0116_tkl.kicad_pcb (KiCad board)
At the start: 2 copper layers, 277.7 x 113.8 mm, 160 parts, among them J1 LiPo, J2 TrackPoint, J3 USB-C (case), J4 USB-C (to nice!nano), SW1 Reset, SW2 Battery, U1 nice!nano_v2, U2 74HC595, U3 74HC595, U5 MCP1700-3302E/TO

Commit message: Route TKL board, add GND stitching, TODO and bilingual READMEs
- m0116_tkl.kicad_pcb: Freerouting result imported; open are only
  GND at J2 pin 2, col2 at U2 pin 1 and the USB daughterboard (tab
  outline still to be sized)
- export_matrix_dsn.py: --continue routes GND as tracks with signal
  width, USB daughterboard nets left out, outline shrunk / holes
  enlarged for KiCad's 0.5 mm edge clearance
- tools/stitch_gnd.py: vias from GND pour islands to the main pour
- TODO.md: remaining steps for KiCad beginners
- README.md and firmware/qmk/readme.md in German and English

Co-Authored-By: Claude Opus 5.5 <noreply@anthropic.com>
Routing:
- net GND: track 0.00 -> 354.7 mm, vias 2 -> 15
- net row1: track 335.5 -> 336.8 mm
